File: FluxGuard-v3.0.kicad_pcb (KiCad board)
At the start: 4 copper layers, 52 x 29 mm, 0 parts

Commit message: Use KiCad 5.99/6.0 compatible format
Other:
- copper layers 4 -> 2
- net class Default: clearance 0.15 -> 0.2; trace_width 0.2 -> 0.25; via_dia 0.6 -> 0.8; via_drill 0.3 -> 0.4
- net class Power removed
Changed lines of the file:
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@@
-(kicad_pcb (version 20221018) (host pcbnew 7.0.0)
+(kicad_pcb (version 20211014) (host pcbnew "(5.99.0)")
   (general
     (thickness 1.6)
-    (legacy_teardrops no)
   )
   (paper "A4")
@@
   )
   (layers
-    (0 "F.Cu" signal)
-    (1 "In1.Cu" power)
-    (2 "In2.Cu" power)
-    (31 "B.Cu" signal)
-    (32 "B.Adhes" user "B.Adhesive")
-    (33 "F.Adhes" user "F.Adhesive")
-    (34 "B.Paste" user)
-    (35 "F.Paste" user)
-    (36 "B.SilkS" user "B.Silkscreen")
-    (37 "F.SilkS" user "F.Silkscreen")
-    (38 "B.Mask" user)
-    (39 "F.Mask" user)
-    (40 "Dwgs.User" user "User.Drawings")
-    (41 "Cmts.User" user "User.Comments")
-    (42 "Eco1.User" user "User.Eco1")
-    (43 "Eco2.User" user "User.Eco2")
-    (44 "Edge.Cuts" user)
-    (45 "Margin" user)
-    (46 "B.CrtYd" user "B.Courtyard")
-    (47 "F.CrtYd" user "F.Courtyard")
-    (48 "B.Fab" user)
-    (49 "F.Fab" user)
+    (0 F.Cu signal)
+    (31 B.Cu signal)
+    (32 B.Adhes user)
+    (33 F.Adhes user)
+    (34 B.Paste user)
+    (35 F.Paste user)
+    (36 B.SilkS user)
+    (37 F.SilkS user)
+    (38 B.Mask user)
+    (39 F.Mask user)
+    (40 Dwgs.User user)
+    (41 Cmts.User user)
+    (42 Eco1.User user)
+    (43 Eco2.User user)
+    (44 Edge.Cuts user)
+    (45 Margin user)
+    (46 B.CrtYd user)
+    (47 F.CrtYd user)
+    (48 B.Fab user)
+    (49 F.Fab user)
   )
   (setup
+    (last_trace_width 0.25)
+    (trace_clearance 0.2)
+    (zone_clearance 0.508)
+    (zone_45_only no)
+    (trace_min 0.2)
+    (via_size 0.8)
+    (via_drill 0.4)
+    (via_min_size 0.4)
+    (via_min_drill 0.3)
+    (uvia_size 0.3)
+    (uvia_drill 0.1)
+    (uvias_allowed no)
+    (uvia_min_size 0.2)
+    (uvia_min_drill 0.1)
+    (edge_width 0.05)
+    (segment_width 0.2)
+    (pcb_text_width 0.3)
+    (pcb_text_size 1.5 1.5)
+    (mod_edge_width 0.12)
+    (mod_text_size 1 1)
+    (mod_text_width 0.15)
+    (pad_size 1.524 1.524)
+    (pad_drill 0.762)
     (pad_to_mask_clearance 0.05)
-    (allow_soldermask_bridges_in_footprints no)
-    (pcbplotparams
-      (layerselection 0x00010fc_ffffffff)
-      (plot_on_all_layers_selection 0x0000000_00000000)
-      (disableapertmacros no)
-      (usegerberextensions yes)
-      (usegerberattributes yes)
-      (usegerberadvancedattributes yes)
-      (creategerberjobfile yes)
-      (dashed_line_dash_ratio 12.000000)
-      (dashed_line_gap_ratio 3.000000)
-      (svgprecision 6)
-      (svgprecision 4)
-      (excludeedgelayer yes)
-      (plotframeref no)
-      (viasonmask no)
-      (mode 1)
-      (useauxorigin no)
-      (hpglpennumber 1)
-      (hpglpenspeed 20)
-      (hpglpendiameter 15.000000)
-      (dxfpolygonmode yes)
-      (dxfimperialunits yes)
-      (dxfusepcbnewfont yes)
-      (psnegative no)
-      (psa4output no)
-      (plotreference yes)
-      (plotvalue yes)
-      (plotinvisibletext no)
-      (sketchpadsonfab no)
-      (subtractmaskfromsilk no)
-      (outputformat 1)
-      (mirror no)
-      (drillshape 0)
-      (scaleselection 1)
-      (outputdirectory "gerber/")
-    )
+    (aux_axis_origin 0 0)
   )
   (net 0 "")
-  (net_class "Default" ""
-    (clearance 0.15)
-    (trace_width 0.2)
-    (via_dia 0.6)
-    (via_drill 0.3)
+  (net_class Default ""
+    (clearance 0.2)
+    (trace_width 0.25)
+    (via_dia 0.8)
+    (via_drill 0.4)
     (uvia_dia 0.3)
     (uvia_drill 0.1)
   )
-  (net_class "Power" ""
-    (clearance 0.2)
-    (trace_width 0.4)
-    (via_dia 0.8)
-    (via_drill 0.4)
-  )
-  (gr_rect (start 0 0) (end 52 29) (stroke (width 0.15) (type solid)) (fill none) (layer "Edge.Cuts"))
+  (gr_line (start 0 0) (end 52 0) (layer Edge.Cuts) (width 0.15))
+  (gr_line (start 52 0) (end 52 29) (layer Edge.Cuts) (width 0.15))
+  (gr_line (start 52 29) (end 0 29) (layer Edge.Cuts) (width 0.15))
+  (gr_line (start 0 29) (end 0 0) (layer Edge.Cuts) (width 0.15))
 )

Commit message: Update to KiCad 9.0 format (version 20240108)
Other:
- copper layers 2 -> 4
Changed lines of the file:
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@@
-(kicad_pcb (version 20211014) (host pcbnew "(5.99.0)")
+(kicad_pcb
+  (version 20240108)
+  (generator "pcbnew")
   (general
     (thickness 1.6)
+    (legacy_teardrops no)
   )
   (paper "A4")
@@
   )
   (layers
-    (0 F.Cu signal)
-    (31 B.Cu signal)
-    (32 B.Adhes user)
-    (33 F.Adhes user)
-    (34 B.Paste user)
-    (35 F.Paste user)
-    (36 B.SilkS user)
-    (37 F.SilkS user)
-    (38 B.Mask user)
-    (39 F.Mask user)
-    (40 Dwgs.User user)
-    (41 Cmts.User user)
-    (42 Eco1.User user)
-    (43 Eco2.User user)
-    (44 Edge.Cuts user)
-    (45 Margin user)
-    (46 B.CrtYd user)
-    (47 F.CrtYd user)
-    (48 B.Fab user)
-    (49 F.Fab user)
+    (0 "F.Cu" signal)
+    (1 "In1.Cu" signal)
+    (2 "In2.Cu" signal)
+    (31 "B.Cu" signal)
+    (32 "B.Adhes" user "B.Adhesive")
+    (33 "F.Adhes" user "F.Adhesive")
+    (34 "B.Paste" user)
+    (35 "F.Paste" user)
+    (36 "B.SilkS" user "B.Silkscreen")
+    (37 "F.SilkS" user "F.Silkscreen")
+    (38 "B.Mask" user)
+    (39 "F.Mask" user)
+    (40 "Dwgs.User" user "User.Drawings")
+    (41 "Cmts.User" user "User.Comments")
+    (42 "Eco1.User" user "User.Eco1")
+    (43 "Eco2.User" user "User.Eco2")
+    (44 "Edge.Cuts" user)
+    (45 "Margin" user)
+    (46 "B.CrtYd" user "B.Courtyard")
+    (47 "F.CrtYd" user "F.Courtyard")
+    (48 "B.Fab" user)
+    (49 "F.Fab" user)
+    (50 "User.1" user)
+    (51 "User.2" user)
+    (52 "User.3" user)
+    (53 "User.4" user)
+    (54 "User.5" user)
+    (55 "User.6" user)
+    (56 "User.7" user)
+    (57 "User.8" user)
+    (58 "User.9" user)
   )
   (setup
-    (last_trace_width 0.25)
-    (trace_clearance 0.2)
-    (zone_clearance 0.508)
-    (zone_45_only no)
-    (trace_min 0.2)
-    (via_size 0.8)
-    (via_drill 0.4)
-    (via_min_size 0.4)
-    (via_min_drill 0.3)
-    (uvia_size 0.3)
-    (uvia_drill 0.1)
-    (uvias_allowed no)
-    (uvia_min_size 0.2)
-    (uvia_min_drill 0.1)
-    (edge_width 0.05)
-    (segment_width 0.2)
-    (pcb_text_width 0.3)
-    (pcb_text_size 1.5 1.5)
-    (mod_edge_width 0.12)
-    (mod_text_size 1 1)
-    (mod_text_width 0.15)
-    (pad_size 1.524 1.524)
-    (pad_drill 0.762)
     (pad_to_mask_clearance 0.05)
-    (aux_axis_origin 0 0)
+    (allow_soldermask_bridges_in_footprints no)
+    (solder_mask_min_width 0.0)
+    (grid_origin 0 0)
+    (drawing_origin 0 0)
   )
   (net 0 "")
-  (net_class Default ""
+  (net_class "Default" ""
     (clearance 0.2)
     (trace_width 0.25)
@@
     (uvia_dia 0.3)
     (uvia_drill 0.1)
+    (diff_pair_gap 0.25)
+    (diff_pair_width 0.2)
   )
-  (gr_line (start 0 0) (end 52 0) (layer Edge.Cuts) (width 0.15))
-  (gr_line (start 52 0) (end 52 29) (layer Edge.Cuts) (width 0.15))
-  (gr_line (start 52 29) (end 0 29) (layer Edge.Cuts) (width 0.15))
-  (gr_line (start 0 29) (end 0 0) (layer Edge.Cuts) (width 0.15))
+  (gr_rect
+    (start 0 0)
+    (end 52 29)
+    (stroke (width 0.15) (type solid))
+    (fill none)
+    (layer "Edge.Cuts")
+  )
 )
