File: FluxGuard-v3.0.kicad_sch (KiCad schematic)
At the start: 70 parts, among them J1 USB_C_Receptacle, J2 TARGET_UART, J3 DEBUG, J4 BATTERY, Q1 FS8205A, SW1 BTN_OK, SW2 BTN_NEXT, SW3 BTN_BACK, U1 ESP32-WROOM-32E, U2 CH340N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

Commit message: Use KiCad 5.99/6.0 compatible format
Parts:
- removed BZ1: MLT-8530, Buzzer_Beeper:Buzzer_MLT-8530, symbol Device:Buzzer
- removed C1, C10, C11, C12, C13, C14, C15, C2, C3, C4, C5, C6, C7, C8, C9: 100nF, Capacitor_SMD:C_0603_1608Metric, symbol Device:C
- removed C16, C17, C18, C19: 10uF, Capacitor_SMD:C_0805_2012Metric, symbol Device:C
- removed C20, C21: 22uF, Capacitor_SMD:C_1206_3216Metric, symbol Device:C
- removed D1: WS2812B-2020, LED_SMD:LED_WS2812B-2020_PLCC4_2.0x2.0mm, symbol LED:WS2812B
- removed D2: PWR_RED, LED_SMD:LED_0603_1608Metric, symbol Device:LED
- removed D3: CHG_YELLOW, LED_SMD:LED_0603_1608Metric, symbol Device:LED
- removed D4: DONE_GREEN, LED_SMD:LED_0603_1608Metric, symbol Device:LED
- removed DISP1: SSD1306_0.96in, Display:OLED_0.96in_128x64_FPC30, symbol Display:SSD1306_OLED_0.96in
- removed J1: USB_C_Receptacle, Connector_USB:USB_C_Receptacle_HRO_TYPE-C-31-M-12_2x6_P0.5mm_Horizontal, symbol Connector:USB_C_Receptacle_USB2.0_16P
- removed J2: TARGET_UART, Connector_PinHeader_2.54mm:PinHeader_2x05_P2.54mm_Vertical, symbol Connector:Conn_01x10_Male
- removed J3: DEBUG, Connector_PinHeader_1.27mm:PinHeader_2x03_P1.27mm_Vertical, symbol Connector:Conn_01x06_Male
- removed J4: BATTERY, Connector_JST:JST_PH_B2B-PH-K_1x02_P2.00mm_Vertical, symbol Connector:Conn_01x02_Male
- removed L1: 2.2uH, Inductor_SMD:L_0805_2012Metric, symbol Device:L
- removed Q1: FS8205A, Package_SO:TSSOP-8_4.4x3mm_P0.65mm, symbol Device:Q_Dual_PMOS_S1G1D2S2G2D1
- removed R1, R10, R2, R3, R4, R5, R6, R7, R8, R9: 10K, Resistor_SMD:R_0603_1608Metric, symbol Device:R
- removed R11, R12: 4.7K, Resistor_SMD:R_0603_1608Metric, symbol Device:R
- removed R13, R14, R15: 100R, Resistor_SMD:R_0603_1608Metric, symbol Device:R
- removed SW1: BTN_OK, Button_Switch_SMD:SW_Push_1P1T_NO_6x6mm_H9.5mm, symbol Switch:SW_Push
- removed SW2: BTN_NEXT, Button_Switch_SMD:SW_Push_1P1T_NO_6x6mm_H9.5mm, symbol Switch:SW_Push
- removed SW3: BTN_BACK, Button_Switch_SMD:SW_Push_1P1T_NO_6x6mm_H9.5mm, symbol Switch:SW_Push
- removed TP1: +3V3, TestPoint:TestPoint_Pad_D1.0mm, symbol Connector:TestPoint
- removed TP2: VBUS, TestPoint:TestPoint_Pad_D1.0mm, symbol Connector:TestPoint
- removed TP3: VBATT, TestPoint:TestPoint_Pad_D1.0mm, symbol Connector:TestPoint
- removed TP4: GND, TestPoint:TestPoint_Pad_D1.0mm, symbol Connector:TestPoint
- removed TP5: I2C_SDA, TestPoint:TestPoint_Pad_D1.0mm, symbol Connector:TestPoint
- removed TP6: I2C_SCL, TestPoint:TestPoint_Pad_D1.0mm, symbol Connector:TestPoint
- removed TP7: TARGET_TX, TestPoint:TestPoint_Pad_D1.0mm, symbol Connector:TestPoint
- removed TP8: TARGET_RX, TestPoint:TestPoint_Pad_D1.0mm, symbol Connector:TestPoint
- removed TVS1, TVS2: SRV05-4, Package_TO_SOT_SMD:SOT-23-6, symbol Device:TVS_4x
- removed U1: ESP32-WROOM-32E, RF_Module:ESP32-WROOM-32, symbol RF_Module:ESP32-WROOM-32E
- removed U2: CH340N, Package_SO:SOIC-8_3.9x4.9mm_P1.27mm, symbol Interface_USB:CH340N
- removed U3: AMS1117-3.3, Package_TO_SOT_SMD:SOT-223-3_TabPin2, symbol Regulator_Linear:AMS1117-3.3
- removed U4: TP4056, Package_SO:SOIC-8_3.9x4.9mm_P1.27mm, symbol Battery_Management:TP4056
- removed U5: DW01A, Package_TO_SOT_SMD:SOT-23-6, symbol Battery_Management:DW01A
- removed U6: ATECC608A, Package_SO:SOIC-8_3.9x4.9mm_P1.27mm, symbol Security:ATECC608A-SSHDA
- removed U7: MAX6818, Package_TO_SOT_SMD:SOT-23-5, symbol Timer:MAX6818
- removed Y1: 26MHz, Oscillator:Oscillator_SMD_3225-4Pin_3.2x2.5mm, symbol Device:Crystal
- removed Y2: 32.768kHz, Crystal:Crystal_SMD_2012-2Pin_2.0x1.2mm, symbol Device:Crystal
- added ?: (no value), symbol power:+3V3
- added ?: (no value), symbol power:GND
- added ?: (no value), symbol power:VBUS
Other:
- company: (none) -> Hangzhou Visularity Technology Co., Ltd.
- title: (none) -> FluxGuard Deployment Dongle v3.0

Commit message: Update to KiCad 9.0 format (version 20240108)
Parts:
- removed ?: (no value), symbol power:+3V3
- removed ?: (no value), symbol power:GND
- removed ?: (no value), symbol power:VBUS
Changed lines of the file:
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@@
-(kicad_sch (version 20211123) (generator eeschema)
+(kicad_sch (version 20231120) (generator "eeschema" (type iter))
+  (version 20231120)
+  (generator "eeschema")
   (paper "A4")
   (title_block
@@
     (company "Hangzhou Visularity Technology Co., Ltd.")
   )
-  (symbol (lib_id "power:+3V3") (at 25.4 20.32 0) (unit 1) (in_bom no) (on_board no) (fields_autoplaced yes)
-  )
-  (symbol (lib_id "power:GND") (at 25.4 25.4 0) (unit 1) (in_bom no) (on_board no) (fields_autoplaced yes)
-  )
-  (symbol (lib_id "power:VBUS") (at 15.24 20.32 0) (unit 1) (in_bom no) (on_board no) (fields_autoplaced yes)
-  )
 )

Commit message: Add schematic with components and wires for KiCad 9
Parts:
- added BZ1: Buzzer, Buzzer_Beeper:Buzzer_12x9.5RM7.6, symbol Device:Buzzer
- added C1, C10, C2, C3, C4, C5, C6, C7, C8, C9: 100nF, Capacitor_SMD:C_0603_1608Metric, symbol Device:C
- added D1: WS2812B, LED_SMD:LED_WS2812B_PLCC4_5.0x5.0mm_P3.2mm, symbol LED:WS2812B
- added J1: USB_C, Connector_USB:USB_C_Receptacle_HRO_TYPE-C-31-M-12, symbol Connector:USB_C_Receptacle_USB2.0_16P
- added J5: OLED_I2C, Connector_PinHeader_2.54mm:PinHeader_1x04_P2.54mm_Vertical, symbol Connector_Generic:Conn_01x04
- added R1, R10, R2, R3, R4, R5, R6, R7, R8, R9: 10K, Resistor_SMD:R_0603_1608Metric, symbol Device:R
- added SW1: BTN_OK, Button_Switch_THT:SW_PUSH_6mm, symbol Switch:SW_Push
- added SW2: BTN_NEXT, Button_Switch_THT:SW_PUSH_6mm, symbol Switch:SW_Push
- added SW3: BTN_BACK, Button_Switch_THT:SW_PUSH_6mm, symbol Switch:SW_Push
- added U1: ESP32-WROOM-32E, RF_Module:ESP32-WROOM-32, symbol RF_Module:ESP32-WROOM-32E
- added U2: CH340N, Package_SO:SOIC-8_3.9x4.9mm_P1.27mm, symbol Interface_USB:CH340N
- added U3: AMS1117-3.3, Package_TO_SOT_SMD:SOT-223-3_TabPin2, symbol Regulator_Linear:AMS1117-3.3
- added U4: TP4056, Package_SO:SOIC-8_3.9x4.9mm_P1.27mm, symbol Battery_Management:TP4056
- added U5: DW01A, Package_TO_SOT_SMD:SOT-23-6, symbol Battery_Management:DW01A
- added U6: ATECC608A, Package_SO:SOIC-8_3.9x4.9mm_P1.27mm, symbol Security:ATECC608A-SSHDA
- added U7: MAX6818, Package_TO_SOT_SMD:SOT-23-5, symbol Timer:MAX6818
Other:
- company: Hangzhou Visularity Technology Co., Ltd. -> (none)
- title: FluxGuard Deployment Dongle v3.0 -> (none)
